Commit message: RL + Hector

File: mini_ros/urdf/accessories.urdf.xacro (robot description, xacro)
@@ -34,4 +34,24 @@
         </plugin>
     </gazebo>
+    <!-- <gazebo reference="imu_link">
+        <gravity>true</gravity>
+        <sensor name="imu_sensor" type="imu">
+        <always_on>true</always_on>
+        <update_rate>100</update_rate>
+        <visualize>true</visualize>
+        <topic>__default_topic__</topic>
+        <plugin filename="libgazebo_ros_imu_sensor.so" name="imu_plugin">
+            <topicName>imu</topicName>
+            <bodyName>imu_link</bodyName>
+            <updateRateHZ>10.0</updateRateHZ>
+            <gaussianNoise>0.0</gaussianNoise>
+            <xyzOffset>0 0 0</xyzOffset>
+            <rpyOffset>0 0 0</rpyOffset>
+            <frameName>imu_link</frameName>
+            <initialOrientationAsReference>false</initialOrientationAsReference>
+        </plugin>
+        <pose>0 0 0 0 0 0</pose>
+        </sensor>
+    </gazebo> -->
     <link name="imu_link">
         <inertial>
@@ -45,4 +65,67 @@
         <child link="imu_link" />
     </joint>
+    <!-- camera -->
+  <gazebo reference="camera">
+    <sensor type="camera" name="camera1">
+      <update_rate>30.0</update_rate>
+      <camera name="head">
+        <horizontal_fov>1.3962634</horizontal_fov>
+        <image>
+          <width>800</width>
+          <height>800</height>
+          <format>R8G8B8</format>
+        </image>
+        <clip>
+          <near>0.02</near>
+          <far>300</far>
+        </clip>
+      </camera>
+      <plugin name="camera_controller" filename="libgazebo_ros_camera.so">
+        <alwaysOn>true</alwaysOn>
+        <updateRate>0.0</updateRate>
+        <cameraName>camera</cameraName>
+        <imageTopicName>rgb/image_raw</imageTopicName>
+        <cameraInfoTopicName>rgb/camera_info</cameraInfoTopicName>
+        <frameName>camera</frameName>
+        <hackBaseline>0.07</hackBaseline>
+        <distortionK1>0.0</distortionK1>
+        <distortionK2>0.0</distortionK2>
+        <distortionK3>0.0</distortionK3>
+        <distortionT1>0.0</distortionT1>
+        <distortionT2>0.0</distortionT2>
+      </plugin>
+    </sensor>
+  </gazebo>
+  <!-- Camera Link -->
+  <link name='camera'>
+    <inertial>
+      <mass value="0.1"/>
+      <origin xyz="0 0 0" rpy=" 0 0 0"/>
+      <inertia
+          ixx="1e-6" ixy="0" ixz="0"
+          iyy="1e-6" iyz="0"
+          izz="1e-6"
+      />
+    </inertial>
+    <collision name='camera_collision'>
+      <origin xyz="0 0 0" rpy=" 0 0 0"/>
+      <geometry>
+        <box size=".01 .01 .01"/>
+      </geometry>
+    </collision>
+    <visual name='camera_visual'>
+      <origin xyz="0 0 0" rpy=" 0 0 0"/>
+      <geometry>
+        <box size=".01 .01 .01"/>
+      </geometry>
+    </visual>
+  </link>
+  <!-- Camera Joint -->
+  <joint type="fixed" name="camera_joint">
+    <origin xyz="0.2 0 0" rpy="0 0 0"/>
+    <child link="camera"/>
+    <parent link="base_link"/>
+    <axis xyz="0 1 0"/>
+  </joint>
     <!-- <xacro:include filename="$(find champ_arm_description)/urdf/champ_arm.urdf.xacro" />
     <xacro:champ_arm parent="base_link">

File: mini_ros/urdf/spot.urdf.xacro (robot description, xacro)
@@ -4,5 +4,5 @@
   <xacro:include filename="$(find mini_ros)/urdf/spot_macro.xacro" />
   <xacro:include filename="$(find mini_ros)/urdf/transmissions.xacro" />
-  <!-- <xacro:include filename="$(find mini_ros)/urdf/accessories.urdf.xacro" /> -->
+  <xacro:include filename="$(find mini_ros)/urdf/accessories.urdf.xacro" />
   <!-- Robot description -->
   <!-- STATIC Links -->

Commit message: Added camera and image processing

File: mini_ros/urdf/accessories.urdf.xacro (robot description, xacro)
@@ -1,5 +1,5 @@
 <?xml version="1.0"?>
 <robot xmlns:xacro="http://ros.org/wiki/xacro">
-    <xacro:include filename="$(find hector_sensors_description)/urdf/hokuyo_utm30lx.urdf.xacro" />
+    <!-- <xacro:include filename="$(find hector_sensors_description)/urdf/hokuyo_utm30lx.urdf.xacro" />
     <xacro:include filename="$(find hector_sensors_description)/urdf/asus_camera.urdf.xacro" />
     <xacro:hokuyo_utm30lx
@@ -15,5 +15,5 @@
     <gazebo reference="hokuyo_frame">
 		<material>Gazebo/FlatBlack</material>
-	</gazebo>
+	</gazebo> -->
     <!-- <xacro:asus_camera
         parent="base_link"
@@ -21,5 +21,5 @@
         <origin xyz="0.2 0.0 0.05" rpy="0 0 0"/>
     </xacro:asus_camera> -->
-    <gazebo>
+    <!-- <gazebo>
         <plugin name="imu_controller" filename="libhector_gazebo_ros_imu.so">
             <updateRate>50.0</updateRate>
@@ -33,8 +33,9 @@
             <headingGaussianNoise>0.005</headingGaussianNoise>
         </plugin>
-    </gazebo>
-    <!-- <gazebo reference="imu_link">
-        <gravity>true</gravity>
-        <sensor name="imu_sensor" type="imu">
+    </gazebo> -->
+  <!-- IMU plugin -->
+  <gazebo reference="imu_link">
+      <gravity>true</gravity>
+      <sensor name="imu_sensor" type="imu">
         <always_on>true</always_on>
         <update_rate>100</update_rate>
@@ -42,5 +43,5 @@
         <topic>__default_topic__</topic>
         <plugin filename="libgazebo_ros_imu_sensor.so" name="imu_plugin">
-            <topicName>imu</topicName>
+            <topicName>imu_data</topicName>
             <bodyName>imu_link</bodyName>
             <updateRateHZ>10.0</updateRateHZ>
@@ -52,20 +53,23 @@
         </plugin>
         <pose>0 0 0 0 0 0</pose>
-        </sensor>
-    </gazebo> -->
-    <link name="imu_link">
-        <inertial>
-            <mass value="0.001"/>
-            <origin xyz="0 0 0" rpy="0 0 0"/>
-            <inertia ixx="1e-09" ixy="0.0" ixz="0.0" iyy="1e-09" iyz="0.0" izz="1e-09"/>
-        </inertial>
-    </link>
-    <joint name="imu_joint" type="fixed">
-        <parent link="base_link" />
-        <child link="imu_link" />
-    </joint>
-    <!-- camera -->
-  <gazebo reference="camera">
-    <sensor type="camera" name="camera1">
+      </sensor>
+  </gazebo>
+  <!-- IMU Link -->
+  <link name="imu_link">
+      <inertial>
+          <mass value="0.001"/>
+          <origin xyz="0 0 0" rpy="0 0 0"/>
+          <inertia ixx="1e-09" ixy="0.0" ixz="0.0" iyy="1e-09" iyz="0.0" izz="1e-09"/>
+      </inertial>
+  </link>
+  <!-- IMU Joint -->
+  <joint name="imu_joint" type="fixed">
+      <parent link="base_link" />
+      <child link="imu_link" />
+  </joint>
+  <!-- Camera Plugin -->
+  <gazebo reference="camera_link">
+    <material>Gazebo/Red</material>
+    <sensor type="camera" name="spot_camera">
       <update_rate>30.0</update_rate>
       <camera name="head">
@@ -84,8 +88,8 @@
         <alwaysOn>true</alwaysOn>
         <updateRate>0.0</updateRate>
-        <cameraName>camera</cameraName>
-        <imageTopicName>rgb/image_raw</imageTopicName>
-        <cameraInfoTopicName>rgb/camera_info</cameraInfoTopicName>
-        <frameName>camera</frameName>
+        <cameraName>spot_camera</cameraName>
+        <imageTopicName>image_raw</imageTopicName>
+        <cameraInfoTopicName>camera_info</cameraInfoTopicName>
+        <frameName>camera_link</frameName>
         <hackBaseline>0.07</hackBaseline>
         <distortionK1>0.0</distortionK1>
@@ -98,5 +102,5 @@
   </gazebo>
   <!-- Camera Link -->
-  <link name='camera'>
+  <link name='camera_link'>
     <inertial>
       <mass value="0.1"/>
@@ -124,5 +128,5 @@
   <joint type="fixed" name="camera_joint">
     <origin xyz="0.2 0 0" rpy="0 0 0"/>
-    <child link="camera"/>
+    <child link="camera_link"/>
     <parent link="base_link"/>
     <axis xyz="0 1 0"/>
